File: vocoder_faceplate/vocoder_faceplate.kicad_pcb (KiCad board)
At the start: 2 copper layers, 121 x 106 mm, 0 parts

Commit message: Add gerber files and images
Other:
- board text added: "Internal Cut Out"
- board text added: "MODULATOR FREQ OFFSET"
- board text removed: "MODULATOR OFFSET"
Changed lines of the file:
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@@
   (general
     (thickness 1.6)
-    (drawings 152)
+    (drawings 162)
     (tracks 0)
     (zones 0)
@@
     (visible_elements 7FFFFFFF)
     (pcbplotparams
-      (layerselection 0x010fc_ffffffff)
+      (layerselection 0x011f0_ffffffff)
       (usegerberextensions false)
       (usegerberattributes false)
@@
       (psa4output false)
       (plotreference true)
-      (plotvalue true)
+      (plotvalue false)
       (plotinvisibletext false)
-      (padsonsilk false)
+      (padsonsilk true)
       (subtractmaskfromsilk false)
       (outputformat 1)
       (mirror false)
-      (drillshape 1)
+      (drillshape 0)
       (scaleselection 1)
-      (outputdirectory ""))
+      (outputdirectory "../gerber/"))
   )
   (net 0 "")
@@
     (uvia_drill 0.1)
   )
-  (gr_circle (center 233 105.5) (end 229 105.5) (layer Dwgs.User) (width 0.15))
-  (gr_line (start 127 148) (end 127 42) (layer Dwgs.User) (width 0.15))
+  (gr_text "Internal Cut Out" (at 165.5 129.5) (layer Dwgs.User)
+    (effects (font (size 1 1) (thickness 0.15)))
+  )
+  (gr_text "Internal Cut Out" (at 138 129.5) (layer Dwgs.User)
+    (effects (font (size 1 1) (thickness 0.15)))
+  )
+  (gr_text "Internal Cut Out" (at 110.5 129.5) (layer Dwgs.User)
+    (effects (font (size 1 1) (thickness 0.15)))
+  )
+  (gr_text "Internal Cut Out" (at 83 129.5) (layer Dwgs.User)
+    (effects (font (size 1 1) (thickness 0.15)))
+  )
+  (gr_text "Internal Cut Out" (at 83 55.5) (layer Dwgs.User)
+    (effects (font (size 1 1) (thickness 0.15)))
+  )
+  (gr_text "Internal Cut Out" (at 165.5 55.5) (layer Dwgs.User)
+    (effects (font (size 1 1) (thickness 0.15)))
+  )
+  (gr_text "Internal Cut Out" (at 138 55.5) (layer Dwgs.User)
+    (effects (font (size 1 1) (thickness 0.15)))
+  )
+  (gr_text "Internal Cut Out" (at 110.5 55.5) (layer Dwgs.User)
+    (effects (font (size 1 1) (thickness 0.15)))
+  )
+  (gr_text "Internal Cut Out" (at 83 89) (layer Dwgs.User)
+    (effects (font (size 1 1) (thickness 0.15)))
+  )
+  (gr_circle (center 165.5 129.5) (end 172.5 129.5) (layer Edge.Cuts) (width 0.05))
+  (gr_circle (center 138 129.5) (end 145 129.5) (layer Edge.Cuts) (width 0.05))
+  (gr_circle (center 110.5 129.5) (end 117.5 129.5) (layer Edge.Cuts) (width 0.05))
+  (gr_circle (center 83 129.5) (end 90 129.5) (layer Edge.Cuts) (width 0.05))
+  (gr_circle (center 83 89) (end 90 89) (layer Edge.Cuts) (width 0.05))
+  (gr_circle (center 165.5 55.5) (end 172.5 55.5) (layer Edge.Cuts) (width 0.05))
+  (gr_circle (center 138 55.5) (end 145 55.5) (layer Edge.Cuts) (width 0.05))
+  (gr_circle (center 110.5 55.5) (end 117.5 55.5) (layer Edge.Cuts) (width 0.05))
+  (gr_circle (center 83 55.5) (end 90 55.5) (layer Edge.Cuts) (width 0.05))
+  (gr_text "Internal Cut Out" (at 111.5 92) (layer Dwgs.User)
+    (effects (font (size 1 1) (thickness 0.15)))
+  )
+  (gr_text "Internal Cut Out" (at 160 92) (layer Dwgs.User)
+    (effects (font (size 1 1) (thickness 0.15)))
+  )
+  (gr_line (start 127 148) (end 127 42) (layer Cmts.User) (width 0.15))
   (gr_text "MODULATOR\nLine Input" (at 172.25 102.5) (layer F.SilkS)
     (effects (font (size 1.2 1.2) (thickness 0.2)))
@@
     (effects (font (size 1.2 1.2) (thickness 0.2)))
   )
-  (gr_line (start 166 86) (end 171 86) (layer Dwgs.User) (width 0.15))
-  (gr_line (start 153.5 86) (end 158.5 86) (layer Dwgs.User) (width 0.15))
+  (gr_line (start 166 86) (end 171 86) (layer Cmts.User) (width 0.15))
+  (gr_line (start 153.5 86) (end 158.5 86) (layer Cmts.User) (width 0.15))
   (gr_line (start 171 86) (end 178.5 86) (layer Edge.Cuts) (width 0.05))
   (gr_line (start 171 80) (end 171 86) (layer Edge.Cuts) (width 0.05))
@@
     (effects (font (size 2 2) (thickness 0.3)) (justify left))
   )
-  (gr_line (start 166 86) (end 166 98.5) (layer Dwgs.User) (width 0.15))
-  (gr_line (start 111.5 86) (end 111.5 98.5) (layer Dwgs.User) (width 0.15))
-  (gr_line (start 153.5 86) (end 153.5 98.5) (layer Dwgs.User) (width 0.15))
+  (gr_line (start 166 86) (end 166 98.5) (layer Cmts.User) (width 0.15))
+  (gr_line (start 111.5 86) (end 111.5 98.5) (layer Cmts.User) (width 0.15))
+  (gr_line (start 153.5 86) (end 153.5 98.5) (layer Cmts.User) (width 0.15))
   (gr_text BANDS (at 165.75 141.5) (layer F.SilkS)
     (effects (font (size 2 2) (thickness 0.3)))
@@
     (effects (font (size 2 2) (thickness 0.3)))
   )
-  (gr_text "MODULATOR\nOFFSET" (at 83.25 102.5) (layer F.SilkS)
+  (gr_text "MODULATOR\nFREQ OFFSET" (at 83.25 102.5) (layer F.SilkS)
     (effects (font (size 2 2) (thickness 0.3)))
   )
@@
     (effects (font (size 2 2) (thickness 0.3)))
   )
-  (gr_circle (center 83 129.5) (end 90 129.5) (layer Edge.Cuts) (width 0.05))
-  (gr_circle (center 110.5 129.5) (end 117.5 129.5) (layer Edge.Cuts) (width 0.05))
-  (gr_circle (center 138 129.5) (end 145 129.5) (layer Edge.Cuts) (width 0.05))
-  (gr_circle (center 165.5 129.5) (end 172.5 129.5) (layer Edge.Cuts) (width 0.05))
-  (gr_circle (center 165.5 55.5) (end 172.5 55.5) (layer Edge.Cuts) (width 0.05))
-  (gr_circle (center 138 55.5) (end 145 55.5) (layer Edge.Cuts) (width 0.05))
-  (gr_circle (center 110.5 55.5) (end 117.5 55.5) (layer Edge.Cuts) (width 0.05))
-  (gr_circle (center 83 55.5) (end 90 55.5) (layer Edge.Cuts) (width 0.05))
-  (gr_circle (center 83 89) (end 90 89) (layer Edge.Cuts) (width 0.05))
   (gr_line (start 141 86) (end 141 98.5) (layer Edge.Cuts) (width 0.05))
   (gr_line (start 153.5 86) (end 141 86) (layer Edge.Cuts) (width 0.05))

Commit message: Switch to KiCAD6
Other:
- net class Default removed
